File: pcb/DCBox/DCBox.kicad_sch (KiCad schematic)
At the start: 76 parts, among them J1 Out-1, J2 Out-2, J3 Out-3, J4 DC-IN, J5 Out-4, J6 USB_A, J7 USB_A, J8 Conn_01x04, SW1 SW_Push, U1 MT2492, U2 662K, U3 STC8H1K08_TSSOP20

Commit message: 1. 布局基本完成
Parts:
- added H1, H2, H3, H4: MountingHole, MountingHole:MountingHole_2.2mm_M2, symbol Mechanical:MountingHole
Changed lines of the file:
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@@
     (pin "2")
+  )
+  (symbol (lib_id "Mechanical:MountingHole") (at 196.85 255.27 0) (unit 1)
+    (in_bom yes) (on_board yes) (fields_autoplaced)
+    (property "Reference" "H1" (id 0) (at 199.39 253.9999 0)
+      (effects (font (size 1.27 1.27)) (justify left))
+    )
+    (property "Value" "MountingHole" (id 1) (at 199.39 256.5399 0)
+      (effects (font (size 1.27 1.27)) (justify left))
+    )
+    (property "Footprint" "MountingHole:MountingHole_2.2mm_M2" (id 2) (at 196.85 255.27 0)
+      (effects (font (size 1.27 1.27)) hide)
+    )
+    (property "Datasheet" "~" (id 3) (at 196.85 255.27 0)
+      (effects (font (size 1.27 1.27)) hide)
+    )
   )
   (symbol (lib_id "Device:C_Small") (at 195.58 43.18 0) (unit 1)
@@
     (pin "1")
     (pin "2")
+  )
+  (symbol (lib_id "Mechanical:MountingHole") (at 196.85 261.62 0) (unit 1)
+    (in_bom yes) (on_board yes) (fields_autoplaced)
+    (property "Reference" "H2" (id 0) (at 199.39 260.3499 0)
+      (effects (font (size 1.27 1.27)) (justify left))
+    )
+    (property "Value" "MountingHole" (id 1) (at 199.39 262.8899 0)
+      (effects (font (size 1.27 1.27)) (justify left))
+    )
+    (property "Footprint" "MountingHole:MountingHole_2.2mm_M2" (id 2) (at 196.85 261.62 0)
+      (effects (font (size 1.27 1.27)) hide)
+    )
+    (property "Datasheet" "~" (id 3) (at 196.85 261.62 0)
+      (effects (font (size 1.27 1.27)) hide)
+    )
   )
   (symbol (lib_id "Device:R_Small") (at 254 113.03 0) (unit 1)
@@
     )
     (pin "1")
+  )
+  (symbol (lib_id "Mechanical:MountingHole") (at 196.85 274.32 0) (unit 1)
+    (in_bom yes) (on_board yes) (fields_autoplaced)
+    (property "Reference" "H4" (id 0) (at 199.39 273.0499 0)
+      (effects (font (size 1.27 1.27)) (justify left))
+    )
+    (property "Value" "MountingHole" (id 1) (at 199.39 275.5899 0)
+      (effects (font (size 1.27 1.27)) (justify left))
+    )
+    (property "Footprint" "MountingHole:MountingHole_2.2mm_M2" (id 2) (at 196.85 274.32 0)
+      (effects (font (size 1.27 1.27)) hide)
+    )
+    (property "Datasheet" "~" (id 3) (at 196.85 274.32 0)
+      (effects (font (size 1.27 1.27)) hide)
+    )
   )
   (symbol (lib_id "power:PWR_FLAG") (at 195.58 33.02 0) (unit 1)
@@
     (pin "1")
   )
+  (symbol (lib_id "Mechanical:MountingHole") (at 196.85 267.97 0) (unit 1)
+    (in_bom yes) (on_board yes) (fields_autoplaced)
+    (property "Reference" "H3" (id 0) (at 199.39 266.6999 0)
+      (effects (font (size 1.27 1.27)) (justify left))
+    )
+    (property "Value" "MountingHole" (id 1) (at 199.39 269.2399 0)
+      (effects (font (size 1.27 1.27)) (justify left))
+    )
+    (property "Footprint" "MountingHole:MountingHole_2.2mm_M2" (id 2) (at 196.85 267.97 0)
+      (effects (font (size 1.27 1.27)) hide)
+    )
+    (property "Datasheet" "~" (id 3) (at 196.85 267.97 0)
+      (effects (font (size 1.27 1.27)) hide)
+    )
+  )
   (symbol (lib_id "power:GND") (at 46.99 261.62 270) (unit 1)
     (in_bom yes) (on_board yes)
@@
       (reference "D7") (unit 1) (value "LED") (footprint "lc_lib:0603_LED_N1")
     )
+    (path "/6a3f7144-558f-4a3c-a5c5-c74bbe8cbaf0"
+      (reference "H1") (unit 1) (value "MountingHole") (footprint "MountingHole:MountingHole_2.2mm_M2")
+    )
+    (path "/71f18bbc-30c3-4a1b-b186-2a032053c781"
+      (reference "H2") (unit 1) (value "MountingHole") (footprint "MountingHole:MountingHole_2.2mm_M2")
+    )
+    (path "/fbca894a-649f-401e-a7f0-3653d82cdd60"
+      (reference "H3") (unit 1) (value "MountingHole") (footprint "MountingHole:MountingHole_2.2mm_M2")
+    )
+    (path "/9d5e7326-5602-45d9-bc0c-50e49c008da2"
+      (reference "H4") (unit 1) (value "MountingHole") (footprint "MountingHole:MountingHole_2.2mm_M2")
+    )
     (path "/3546385e-ca55-45e8-bbf6-9c53933ea28a"

Commit message: 1. 布线
Connections:
- net GND: now also C11.2, C12.2
- net SCL: now also U3.1 (P1.2); no longer U3.2 (P1.3)
- net SDA: now also U3.2 (P1.3); no longer U3.1 (P1.2)
- net at J6.4 (GND), J6.5 (Shield), R15.1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: no longer C11.2
- net at J7.4 (GND), J7.5 (Shield), R16.1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: no longer C12.2
Changed lines of the file:
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@@
 (kicad_sch (version 20211123) (generator eeschema)
   (paper "A3")
+  (junction (at 138.43 193.04) (diameter 0) (color 0 0 0 0)
+  )
   (junction (at 66.04 256.54) (diameter 0) (color 0 0 0 0)
   )
@@
   (junction (at 96.52 193.04) (diameter 0) (color 0 0 0 0)
   )
-  (junction (at 110.49 154.94) (diameter 0) (color 0 0 0 0)
-  )
   (junction (at 186.69 49.53) (diameter 0) (color 0 0 0 0)
   )
@@
   (junction (at 186.69 59.69) (diameter 0) (color 0 0 0 0)
   )
+  (junction (at 137.16 154.94) (diameter 0) (color 0 0 0 0)
+  )
   (junction (at 39.37 119.38) (diameter 0) (color 0 0 0 0)
   )
@@
   )
   (junction (at 49.53 261.62) (diameter 0) (color 0 0 0 0)
-  )
-  (junction (at 111.76 193.04) (diameter 0) (color 0 0 0 0)
   )
   (junction (at 359.41 128.27) (diameter 0) (color 0 0 0 0)
@@
     (stroke (width 0) (type default) (color 0 0 0 0))
   )
+  (wire (pts (xy 138.43 198.12) (xy 138.43 193.04))
+    (stroke (width 0) (type default) (color 0 0 0 0))
+  )
   (wire (pts (xy 87.63 223.52) (xy 93.98 223.52))
     (stroke (width 0) (type default) (color 0 0 0 0))
@@
     (stroke (width 0) (type default) (color 0 0 0 0))
   )
+  (wire (pts (xy 137.16 161.29) (xy 137.16 154.94))
+    (stroke (width 0) (type default) (color 0 0 0 0))
+  )
   (wire (pts (xy 346.71 203.2) (xy 356.87 203.2))
     (stroke (width 0) (type default) (color 0 0 0 0))
@@
     (stroke (width 0) (type default) (color 0 0 0 0))
   )
+  (wire (pts (xy 137.16 154.94) (xy 139.7 154.94))
+    (stroke (width 0) (type default) (color 0 0 0 0))
+  )
   (wire (pts (xy 280.67 191.77) (xy 294.64 191.77))
     (stroke (width 0) (type default) (color 0 0 0 0))
@@
     (stroke (width 0) (type default) (color 0 0 0 0))
   )
-  (wire (pts (xy 106.68 198.12) (xy 111.76 198.12))
+  (wire (pts (xy 106.68 198.12) (xy 138.43 198.12))
     (stroke (width 0) (type default) (color 0 0 0 0))
   )
@@
     (stroke (width 0) (type default) (color 0 0 0 0))
   )
-  (wire (pts (xy 106.68 154.94) (xy 110.49 154.94))
-    (stroke (width 0) (type default) (color 0 0 0 0))
-  )
-  (wire (pts (xy 133.35 193.04) (xy 140.97 193.04))
+  (wire (pts (xy 133.35 193.04) (xy 138.43 193.04))
     (stroke (width 0) (type default) (color 0 0 0 0))
   )
@@
     (stroke (width 0) (type default) (color 0 0 0 0))
   )
-  (wire (pts (xy 133.35 154.94) (xy 139.7 154.94))
+  (wire (pts (xy 133.35 154.94) (xy 137.16 154.94))
     (stroke (width 0) (type default) (color 0 0 0 0))
   )
@@
     (stroke (width 0) (type default) (color 0 0 0 0))
   )
-  (wire (pts (xy 111.76 198.12) (xy 111.76 193.04))
-    (stroke (width 0) (type default) (color 0 0 0 0))
-  )
   (wire (pts (xy 280.67 187.96) (xy 294.64 187.96))
     (stroke (width 0) (type default) (color 0 0 0 0))
@@
     (stroke (width 0) (type default) (color 0 0 0 0))
   )
-  (wire (pts (xy 106.68 193.04) (xy 111.76 193.04))
+  (wire (pts (xy 106.68 193.04) (xy 118.11 193.04))
     (stroke (width 0) (type default) (color 0 0 0 0))
   )
@@
     (stroke (width 0) (type default) (color 0 0 0 0))
   )
-  (wire (pts (xy 110.49 161.29) (xy 110.49 154.94))
-    (stroke (width 0) (type default) (color 0 0 0 0))
-  )
   (wire (pts (xy 153.67 26.67) (xy 158.75 26.67))
     (stroke (width 0) (type default) (color 0 0 0 0))
@@
     (stroke (width 0) (type default) (color 0 0 0 0))
   )
-  (wire (pts (xy 110.49 154.94) (xy 118.11 154.94))
+  (wire (pts (xy 106.68 154.94) (xy 118.11 154.94))
     (stroke (width 0) (type default) (color 0 0 0 0))
   )
@@
     (stroke (width 0) (type default) (color 0 0 0 0))
   )
+  (wire (pts (xy 138.43 193.04) (xy 140.97 193.04))
+    (stroke (width 0) (type default) (color 0 0 0 0))
+  )
   (wire (pts (xy 118.11 152.4) (xy 118.11 154.94))
     (stroke (width 0) (type default) (color 0 0 0 0))
@@
     (stroke (width 0) (type default) (color 0 0 0 0))
   )
-  (wire (pts (xy 106.68 161.29) (xy 110.49 161.29))
+  (wire (pts (xy 106.68 161.29) (xy 137.16 161.29))
     (stroke (width 0) (type default) (color 0 0 0 0))
   )
@@
   )
   (wire (pts (xy 154.94 49.53) (xy 175.26 49.53))
-    (stroke (width 0) (type default) (color 0 0 0 0))
-  )
-  (wire (pts (xy 111.76 193.04) (xy 118.11 193.04))
     (stroke (width 0) (type default) (color 0 0 0 0))
   )
@@
     (effects (font (size 1.27 1.27)) (justify right bottom))
   )
-  (label "SCL" (at 237.49 184.15 180)
+  (label "SCL" (at 237.49 180.34 180)
     (effects (font (size 1.27 1.27)) (justify right bottom))
   )
@@
     (effects (font (size 1.27 1.27)) (justify left bottom))
   )
-  (label "SDA" (at 237.49 180.34 180)
+  (label "SDA" (at 237.49 184.15 180)
     (effects (font (size 1.27 1.27)) (justify right bottom))
   )

Commit message: 1. PCB基本完成
Connections:
- net LED_DC1: now also U3.18 (P3.7/TxD2); no longer U3.3 (P1.4)
- net LED_DC2: now also U3.3 (P1.4); no longer U3.4 (P1.5)
- net LED_DC3: now also U3.4 (P1.5); no longer U3.5 (P1.6/RxD_3)
- net LED_DC4: now also U3.5 (P1.6/RxD_3); no longer U3.6 (P1.7/TxD_3)
- net LED_USB1: now also U3.6 (P1.7/TxD_3); no longer U3.7 (P5.4)
- net LED_USB2: now also U3.7 (P5.4); no longer U3.18 (P3.7/TxD2)
Changed lines of the file:
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@@
     (effects (font (size 1.27 1.27)) (justify right bottom))
   )
-  (label "LED_DC4" (at 237.49 199.39 180)
+  (label "LED_DC4" (at 237.49 195.58 180)
     (effects (font (size 1.27 1.27)) (justify right bottom))
   )
@@
     (effects (font (size 1.27 1.27)) (justify left bottom))
   )
-  (label "LED_DC3" (at 237.49 195.58 180)
+  (label "LED_DC3" (at 237.49 191.77 180)
     (effects (font (size 1.27 1.27)) (justify right bottom))
   )
@@
     (effects (font (size 1.27 1.27)) (justify right bottom))
   )
-  (label "LED_USB2" (at 294.64 187.96 0)
-    (effects (font (size 1.27 1.27)) (justify left bottom))
+  (label "LED_USB2" (at 237.49 203.2 180)
+    (effects (font (size 1.27 1.27)) (justify right bottom))
   )
   (label "LED_DC3" (at 243.84 133.35 270)
@@
     (effects (font (size 1.27 1.27)) (justify left bottom))
   )
-  (label "LED_USB1" (at 237.49 203.2 180)
+  (label "LED_USB1" (at 237.49 199.39 180)
     (effects (font (size 1.27 1.27)) (justify right bottom))
   )
@@
     (effects (font (size 1.27 1.27)) (justify left bottom))
   )
-  (label "LED_DC1" (at 237.49 187.96 180)
+  (label "LED_DC1" (at 294.64 187.96 0)
+    (effects (font (size 1.27 1.27)) (justify left bottom))
+  )
+  (label "LED_DC2" (at 237.49 187.96 180)
     (effects (font (size 1.27 1.27)) (justify right bottom))
   )
-  (label "LED_DC2" (at 237.49 191.77 180)
-    (effects (font (size 1.27 1.27)) (justify right bottom))
-  )
